File: Design/Z31_SWC_Rev1/Z31_SWC_Rev1.kicad_pcb (KiCad board)
At the start: 2 copper layers, 69.1 x 46.2 mm, 45 parts, among them J1 Conn_01x16, J2 ICSP, J3 UART, U1 4066, U2 ATMEGA328-AURCT-ND, U3 MCP2510, U4 TJR1443, U5 ULN2003, U6 74HCT164, U7 4066, U8 MMPQ2907A, Y1 16Mhz, Y2 8MHz

Commit message: Final Rev1 design
Parts:
- removed the U3 at (144.0, 113.0)
- added C13: 1u, Capacitor_SMD:C_1210_3225Metric_Pad1.33x2.70mm_HandSolder, F.Cu at (130.1, 83.6)
- added C14: 100nF, Capacitor_SMD:C_0805_2012Metric_Pad1.18x1.45mm_HandSolder, F.Cu at (132.8, 82.8)
- added C15: 22uF, Capacitor_SMD:CP_Elec_5x5.7, F.Cu at (124.0, 82.7)
- added C16: N/A, Capacitor_SMD:C_0805_2012Metric_Pad1.18x1.45mm_HandSolder, F.Cu at (128.7, 88.0)
- added C17: 100nF, Capacitor_SMD:C_0805_2012Metric_Pad1.18x1.45mm_HandSolder, F.Cu at (120.9, 110.5)
- added C18: yes, Capacitor_SMD:C_1210_3225Metric_Pad1.33x2.70mm_HandSolder, F.Cu at (131.2, 91.5)
- added C3: 10uF, Capacitor_SMD:CP_Elec_5x5.7, F.Cu at (147.8, 95.5)
- added D2: D_Schottky, Diode_SMD:D_SMA, F.Cu at (116.9, 84.1)
- added D3: SMAJ18CAQ-13-F, Diode_SMD:D_SMA, F.Cu at (116.9, 80.5)
- added D4: 1N4148, Diode_SMD:D_SOD-323_HandSoldering, F.Cu at (121.8, 93.3)
- added D5: 1N4148, Diode_SMD:D_SOD-323_HandSoldering, F.Cu at (122.9, 97.1)
- added F1: Polyfuse, Fuse:Fuse_1812_4532Metric_Pad1.30x3.40mm_HandSolder, F.Cu at (111.3, 82.7)
- added JP3: Volume_Pull, Jumper:SolderJumper-3_P1.3mm_Open_RoundedPad1.0x1.5mm_NumberLabels, F.Cu at (126.2, 109.9)
- added R10: 1K, Resistor_SMD:R_0805_2012Metric_Pad1.20x1.40mm_HandSolder, F.Cu at (174.7, 104.4)
- added R11: 10k, Resistor_SMD:R_0805_2012Metric_Pad1.20x1.40mm_HandSolder, F.Cu at (142.8, 119.1)
- added R16: 10k, Resistor_SMD:R_0805_2012Metric_Pad1.20x1.40mm_HandSolder, F.Cu at (143.6, 92.3)
- added R21: R_Small, Resistor_SMD:R_0805_2012Metric_Pad1.20x1.40mm_HandSolder, F.Cu at (122.9, 110.5)
- added R22: 10k, Resistor_SMD:R_0805_2012Metric_Pad1.20x1.40mm_HandSolder, F.Cu at (130.3, 106.8)
- added R23: 10k, Resistor_SMD:R_0805_2012Metric_Pad1.20x1.40mm_HandSolder, F.Cu at (128.4, 104.3)
- added R24: 10k, Resistor_SMD:R_0805_2012Metric_Pad1.20x1.40mm_HandSolder, F.Cu at (130.3, 101.8)
- added R25: 10k, Resistor_SMD:R_0805_2012Metric_Pad1.20x1.40mm_HandSolder, F.Cu at (128.4, 99.3)
- added R26: N/A, Resistor_SMD:R_0805_2012Metric_Pad1.20x1.40mm_HandSolder, F.Cu at (130.8, 88.0)
- added R27: N/A, Resistor_SMD:R_0805_2012Metric_Pad1.20x1.40mm_HandSolder, F.Cu at (132.8, 86.7)
- added U5: MCP2515-xST, Package_SO:TSSOP-20_4.4x6.5mm_P0.65mm, F.Cu at (145.8, 104.1)
- added U8: NCV4276B, Package_TO_SOT_SMD:TO-263-5_TabPin3, F.Cu at (142.1, 85.7)
- D1: value 1N4148 -> LED; footprint Diode_SMD:D_SOD-323 -> LED_SMD:LED_0805_2012Metric
- TH1: value THERMISTOR NTC 47K -> NTC 47K
- U6: renamed from U4; footprint Package_SO:SOIC-14_3.9x8.7mm_P1.27mm -> Package_SO:SO-14_3.9x8.65mm_P1.27mm
- moved R2 52.4 mm to (125.6, 93.3), turned to 0 degrees
- moved R3 49.9 mm to (125.7, 91.3)
- moved JP2 35.8 mm to (120.5, 117.0), turned to 0 degrees
- moved U7 33.2 mm to (131.3, 116.9), turned to 90 degrees
- moved JP1 32.2 mm to (124.4, 117.0), turned to 0 degrees
- moved D1 21.8 mm to (146.6, 119.1), turned to 180 degrees
- moved R9 18.8 mm to (151.8, 100.4), turned to -90 degrees
- moved R17 18.5 mm to (130.7, 110.8), turned to -90 degrees
- moved R8 17.0 mm to (158.4, 117.1)
- moved C8 14.2 mm to (146.2, 114.2), turned to 0 degrees
- moved TH1 13.8 mm to (151.1, 119.3), turned to 180 degrees
- moved R18 13.6 mm to (132.3, 105.7), turned to -90 degrees
- moved R19 12.2 mm to (133.2, 102.8), turned to 0 degrees
- moved U4 10.3 mm to (158.2, 92.5)
- moved U1 10.3 mm to (169.6, 92.6)
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- renumbered C3 to C10, C8 to C12, C5 to C4, C6 to C5, C12 to C6, C9 to C7, C10 to C8, C7 to C9, J2 to J1, J3 to J2, J1 to J3, R4 to R1, R11 to R13, R13 to R14, R10 to R15, R14 to R17, R15 to R18, R16 to R19, R5 to R2, R17 to R20, R6 to R3, R1 to R4, R7 to R5, R2 to R6, R3 to R7, U6 to U3, U7 to U4, U5 to U7, U8 to U9
Connections:
- C10 pad 2: +5V -> +12V
- C11 pad 2: +5V -> +12V
- D1 pad 1: /REG_INH -> GND
- J3 pad 1: /+12V_CONST -> GND
- J3 pad 11: /ANALOG_VOL_OUT -> /ASCD_ACCEL
- J3 pad 12: /SWC_OUTPUT_A -> /ASCD_RESUME
- J3 pad 13: /AUX_OUT_1 -> GND
- J3 pad 14: /AUX_OUT_2 -> /SWC_OUTPUT_A
- J3 pad 15: CANH -> /SWC_SIGNAL_IN
- J3 pad 16: CANL -> /AUX_OUT_1
- J3 pad 2: GND -> CANL
- J3 pad 3: /+12V_IGN -> CANH
- J3 pad 5: /SWC_SIGNAL_IN -> /AUX_OUT_2
- J3 pad 6: /+12V_ASCD -> /ASCD_RELAY
- J3 pad 7: /ASCD_RELAY -> /+12V_CONST
- J3 pad 8: /ASCD_RESUME -> Net-(D4-Pad2)
- J3 pad 9: /ASCD_ACCEL -> Net-(D5-Pad2)
- R17 pad 2: Net-(U5-Pad16) -> Net-(R17-Pad2)
- R18 pad 2: Net-(U5-Pad15) -> Net-(R18-Pad2)
- R19 pad 2: Net-(U5-Pad14) -> Net-(R19-Pad2)
- R2 pad 1: +12V -> /+12V_IGN
- R20 pad 2: Net-(U5-Pad13) -> Net-(R20-Pad2)
- U1 pad 14: +5V -> +12V
- U2 pad 1: /CAN_INT -> /A2
- U2 pad 12: /CS_SHIFTOUT -> /CAN_INT
- U2 pad 20: unconnected-(U2-Pad20) -> +5V
- U2 pad 23: unconnected-(U2-Pad23) -> /CR_SET
- U2 pad 24: unconnected-(U2-Pad24) -> /CR_ACCEL
- U2 pad 25: unconnected-(U2-Pad25) -> /CR_RESUME
- U2 pad 26: unconnected-(U2-Pad26) -> /SWC_PWR
- U2 pad 27: unconnected-(U2-Pad27) -> /A1
- U2 pad 28: unconnected-(U2-Pad28) -> /CR_RELAY
- U2 pad 32: /SWC_IN -> /SWC_SIGNAL_IN
- U2 pad 9: unconnected-(U2-Pad9) -> /CS_SHIFTOUT
- U4 pad 14: +5V -> +12V
- U6 pad 7: Net-(D1-Pad2) -> Net-(R16-Pad1)
- U6 pad 8: unconnected-(U4-Pad8) -> /CAN_ERR
- U6 pad 9: unconnected-(U4-Pad9) -> /MODULE_VOLTAGE
- U7 pad 1: unconnected-(U5-Pad1) -> /CR_RELAY
- U7 pad 10: /AUX_2 -> Net-(R20-Pad2)
- U7 pad 11: /AUX_1 -> Net-(R19-Pad2)
- U7 pad 12: /ASCD_RELAY -> Net-(R18-Pad2)
- U7 pad 13: Net-(U5-Pad13) -> Net-(R17-Pad2)
- U7 pad 14: Net-(U5-Pad14) -> /AUX_OUT_2
- U7 pad 15: Net-(U5-Pad15) -> /AUX_1
- U7 pad 16: Net-(U5-Pad16) -> /ASCD_RELAY
- U7 pad 2: unconnected-(U5-Pad2) -> /A1
- U7 pad 3: unconnected-(U5-Pad3) -> /A2
- U7 pad 4: unconnected-(U5-Pad4) -> /SWC_PWR
- U7 pad 5: unconnected-(U5-Pad5) -> /CR_RESUME
- U7 pad 6: unconnected-(U5-Pad6) -> /CR_ACCEL
- U7 pad 7: unconnected-(U5-Pad7) -> /CR_SET
- U7 pad 9: /+12V_CONST -> +12V
- U9 pad 10: /+12V_CONST -> +12V
Routing:
- net +5V: track 19.6 -> 164.4 mm, vias 0 -> 4
- net +12V: track 0.00 -> 139.4 mm, vias 0 -> 4
- net /SWC_OUTPUT_A: track 22.7 -> 145.1 mm
- net /SWC_ANALOG_B: track 65.2 -> 162.6 mm
- net /SWC_SIGNAL_IN: track 0.00 -> 96.8 mm, vias 0 -> 1
- net /MODULE_VOLTAGE: track 0.00 -> 79.6 mm, vias 0 -> 4
- net /A2: track 0.00 -> 72.6 mm
- net /CR_RELAY: track 0.00 -> 69.9 mm, vias 0 -> 2
- net /A1: track 0.00 -> 63.4 mm, vias 0 -> 2
- net /SWC_PWR: track 0.00 -> 61.0 mm
- net /CR_RESUME: track 0.00 -> 57.5 mm
- net /CR_ACCEL: track 0.00 -> 54.9 mm
- net /CR_SET: track 0.00 -> 53.2 mm
- net /RESET: track 0.00 -> 38.9 mm, vias 0 -> 4
- net GND: track 87.6 -> 57.1 mm, vias 10 -> 57
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- added copper zone on B.Cu, net GND
- added copper zone on F.Cu, net GND
- added copper zone on F.Cu, net Net-(D2-Pad2)
Other:
- board text added: "Z31-SWC Rev 1 A.M. 2022"
