File: Design/Z31_SWC_Rev1/Z31_SWC_Rev1.kicad_sch (KiCad schematic)
At the start: 46 parts, among them J1 Conn_01x16, J2 ICSP, J3 UART, U1 4066, U2 ATMEGA328-AURCT-ND, U3 MCP2510, U4 TJR1443, U5 ULN2003, U6 74HCT164, U7 4066, U8 MMPQ2907A, Y1 16Mhz, Y2 8MHz

Commit message: Final Rev1 design
Parts:
- removed D1: 1N4148, Diode_SMD:D_SOD-323, symbol Device:D_Small
- removed U3: MCP2510, Package_SO:TSSOP-20_4.4x6.5mm_P0.65mm, symbol Personal:MCP2510
- added C13: 1u, Capacitor_SMD:C_1210_3225Metric_Pad1.33x2.70mm_HandSolder, symbol Device:C_Small
- added C14, C17: 100nF, Capacitor_SMD:C_0805_2012Metric_Pad1.18x1.45mm_HandSolder, symbol Device:C_Small
- added C15: 22uF, Capacitor_SMD:CP_Elec_5x5.7, symbol Device:C_Polarized_Small
- added C16: N/A, Capacitor_SMD:C_0805_2012Metric_Pad1.18x1.45mm_HandSolder, symbol Device:C_Small
- added C18: yes, Capacitor_SMD:C_1210_3225Metric_Pad1.33x2.70mm_HandSolder, symbol Device:C_Small
- added D1: LED, LED_SMD:LED_0805_2012Metric, symbol Device:LED
- added D2: D_Schottky, Diode_SMD:D_SMA, symbol Device:D_Schottky
- added D3: SMAJ18CAQ-13-F, Diode_SMD:D_SMA, symbol Device:D_TVS
- added D4, D5: 1N4148, Diode_SMD:D_SOD-323_HandSoldering, symbol Device:D_Small
- added F1: Polyfuse, Fuse:Fuse_1812_4532Metric_Pad1.30x3.40mm_HandSolder, symbol Device:Polyfuse
- added JP3: Volume_Pull, Jumper:SolderJumper-3_P1.3mm_Open_RoundedPad1.0x1.5mm_NumberLabels, symbol Jumper:SolderJumper_3_Open
- added R10: 1K, Resistor_SMD:R_0805_2012Metric_Pad1.20x1.40mm_HandSolder, symbol Device:R
- added R11, R16, R22, R23, R24, R25: 10k, Resistor_SMD:R_0805_2012Metric_Pad1.20x1.40mm_HandSolder, symbol Device:R_Small
- added R21: R_Small, Resistor_SMD:R_0805_2012Metric_Pad1.20x1.40mm_HandSolder, symbol Device:R_Small
- added R26, R27: N/A, Resistor_SMD:R_0805_2012Metric_Pad1.20x1.40mm_HandSolder, symbol Device:R_Small
- added U5: MCP2515-xST, Package_SO:TSSOP-20_4.4x6.5mm_P0.65mm, symbol Interface_CAN_LIN:MCP2515-xST
- added U8: NCV4276B, Package_TO_SOT_SMD:TO-263-5_TabPin3, symbol Personal:NCV4276B
- C3: renamed from C4; footprint (none) -> Capacitor_SMD:CP_Elec_5x5.7
- TH1: value THERMISTOR NTC 47K -> NTC 47K
- U6: renamed from U4; footprint Package_SO:SOIC-14_3.9x8.7mm_P1.27mm -> Package_SO:SO-14_3.9x8.65mm_P1.27mm
- renumbered C3 to C10, C8 to C12, C5 to C4, C6 to C5, C12 to C6, C9 to C7, C10 to C8, C7 to C9, J2 to J1, J3 to J2, J1 to J3, R4 to R1, R11 to R13, R13 to R14, R10 to R15, R14 to R17, R15 to R18, R16 to R19, R5 to R2, R17 to R20, R6 to R3, R1 to R4, R7 to R5, R2 to R6, R3 to R7, U6 to U3, U7 to U4, U5 to U7, U8 to U9
Connections:
- net ANALOG_VOL_OUT is gone; now on net ASCD_ACCEL: J3.11 (Pin_11)
- net AUX_2 is gone; now on an unnamed net: U7.10 (O7)
- net SWC_IN is gone; now on net SWC_SIGNAL_IN: U2.32 (PD2)
- net +12V: now also C10.2, C11.2, U1.14 (VDD), U4.14 (VDD), U7.9 (COM), U9.10 (E4), C13.1, C14.1, C15.1, D2.1 (K), JP3.3 (B), R22.2, U8.1 (IN); no longer R2.1
- net +12V_ASCD: now also D5.1 (K), R23.2, R24.2, R25.2; no longer J3.6 (Pin_6)
- net +12V_CONST: now also J3.7 (Pin_7), F1.2; no longer J3.1 (Pin_1), U7.9 (COM), U9.10 (E4)
- net +12V_IGN: now also R2.1, D4.1 (K); no longer J3.3 (Pin_3)
- net +5V: now also U2.20 (AREF), C16.1, C18.1, JP3.1 (A), R10.1, R11.1, R26.1, U5.20 (VDD), U8.5 (OUT); no longer C10.2, C11.2, U1.14 (VDD), U4.14 (VDD)
- net ASCD_ACCEL: no longer J3.9 (Pin_9)
- net ASCD_RELAY: now also J3.6 (Pin_6), U7.16 (O1); no longer J3.7 (Pin_7), U7.12 (O5)
- net ASCD_RESUME: now also J3.12 (Pin_12); no longer J3.8 (Pin_8)
- net AUX_1: now also U7.15 (O2); no longer U7.11 (O6)
- net AUX_OUT_1: now also J3.16 (Pin_16); no longer J3.13 (Pin_13)
- net AUX_OUT_2: now also J3.5 (Pin_5), U7.14 (O3), C17.1, R21.2; no longer J3.14 (Pin_14)
- net CANH: now also J3.3 (Pin_3); no longer J3.15 (Pin_15)
- net CANL: now also J3.2 (Pin_2); no longer J3.16 (Pin_16)
- net CAN_EN: now also U5.12 (~{RX0BF})
- net CAN_INT: now also U2.12 (PB0), U5.13 (~{INT}); no longer U2.1 (PD3)
- net CAN_STB: now also U5.11 (~{RX1BF})
- net CS_CAN: now also U5.18 (~{CS})
- net CS_SHIFTOUT: now also U2.9 (PD5); no longer U2.12 (PB0)
- net GND: now also J3.1 (Pin_1), J3.13 (Pin_13), C13.2, C14.2, C15.2, C17.2, C18.2, D1.1 (K), D3.1 (A1), R16.2, R27.2, U5.10 (VSS), U8.3 (GND); no longer J3.2 (Pin_2)
- net MISO: now also U5.17 (SO)
- net MODULE_VOLTAGE: now also U6.9 (WAKE)
- net MOSI: now also U5.16 (SI)
- net RESET_CAN: now also U5.19 (~{RESET})
- net RXCAN: now also U5.2 (RXCAN)
- net SCK: now also U5.14 (SCK)
- net SWC_OUTPUT_A: now also J3.14 (Pin_14); no longer J3.12 (Pin_12)
- net SWC_SIGNAL_IN: now also J3.15 (Pin_15), R10.2; no longer J3.5 (Pin_5)
- net TXCAN: now also U5.1 (TXCAN)
- net at R20.1, U9.15 (B1): now also R25.1
- net at R20.2: no longer U7.13 (O4)
- net CR_SET: now reaches U2.23 (PC0)
- net CR_SET: now also U7.7 (I7)
- net CR_ACCEL: now reaches U2.24 (PC1)
- net CR_ACCEL: now also U7.6 (I6)
- net CR_RESUME: now reaches U2.25 (PC2)
- net CR_RESUME: now also U7.5 (I5)
- net SWC_PWR: now reaches U2.26 (PC3)
- net SWC_PWR: now also U7.4 (I4)
- net A1: now reaches U2.27 (PC4)
- net A1: now also U7.2 (I2)
- net CR_RELAY: now reaches U2.28 (PC5)
- net CR_RELAY: now also U7.1 (I1)
- net at C7.2, Y2.2: now also U5.8 (OSC2)
- net at C8.2, Y2.1: now also U5.9 (OSC1)
- net at R19.2: now also U7.11 (O6); no longer U7.14 (O3)
- net at R18.2: now also U7.12 (O5); no longer U7.15 (O2)
- net at R17.2: now also U7.13 (O4); no longer U7.16 (O1)
- net A2: now reaches U7.3 (I3)
- net A2: now also U2.1 (PD3)
- net at U6.7 (INH): now also R16.1, U8.2 (~{INH})
- net at R19.1, U9.13 (B2): now also R24.1
- net at R18.1, U9.11 (B3): now also R23.1
- net at R17.1, U9.9 (B4): now also R22.1
- net CAN_ERR: now reaches U6.8 (~{ERR})
- net CAN_ERR: now also U5.4 (~{TX0RTS})
- new net: D4.2 (A), J3.8 (Pin_8)
- new net: D5.2 (A), J3.9 (Pin_9)
- new net: JP3.2 (C), R21.1
- new net: C16.2, R26.2, R27.1, U8.4 (VA)
- new net: D1.2 (A), R11.2
- new net: D2.2 (A), D3.2 (A2), F1.1
Other:
- moved on the sheet: C1, C12, C2, C3, C4, C5, C6, C7, C8, C9, J1, J2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
